Commit message: Addition: Added a python balance controller for the bot.

File: install/self_balancing_bot/share/self_balancing_bot/urdf/robot.urdf.xacro (robot description, xacro)
@@ -90,29 +90,26 @@
   <xacro:wheel name="left" x_offset="0" y_offset="${0.06}"/>
   <xacro:wheel name="right" x_offset="0" y_offset="${-0.06}"/>
-  <link name="camera_link">
-    <visual>
-      <origin xyz="0 0 0.05" rpy="0 0 0"/>
-      <geometry>
-        <box size="0.05 0.05 0.03"/>
-      </geometry>
-      <material name="green">
-        <color rgba="0 0.8 0 1"/>
-      </material>
-    </visual>
-    <collision>
+  <!--Dummy Base Footprint-->
+  <link name="base_footprint"/>
+  <joint name="base_footprint_joint" type="fixed">
+      <parent link="base_footprint"/>
+      <child link="base_link"/>
       <origin xyz="0 0 0" rpy="0 0 0"/>
-      <geometry>
-        <box size="0.05 0.05 0.03"/>
-      </geometry>
-    </collision>
-    <xacro:box_inertia m="0.1" x="0.05" y="0.05" z="0.03" cz="0"/>
-  </link>
-  <joint name="camera_joint" type="fixed">
-    <parent link="base_link"/>
-    <child link="camera_link"/>
-    <!-- Front of robot, tilted down 30 degrees -->
-    <origin xyz="0.08 0 0.12" rpy="0 -0.523 0"/>
   </joint>
   <!--Gazebo_Plugins-->
+  <gazebo>
+    <plugin filename="gz-sim-diff-drive-system"
+            name="gz::sim::systems::DiffDrive">
+      <left_joint>left_wheel_joint</left_joint>
+      <right_joint>right_wheel_joint</right_joint>
+      <wheel_separation>${2 * 0.06}</wheel_separation>
+      <wheel_radius>${wheel_radius}</wheel_radius>
+      <odom_publish_frequency>50</odom_publish_frequency>
+      <topic>/cmd_vel</topic>
+      <odom_topic>/odom</odom_topic>
+      <frame_id>odom</frame_id>
+      <child_frame_id>base_link</child_frame_id>
+    </plugin>
+  </gazebo>
   <gazebo reference="base_link">
     <sensor name="imu_sensor" type="imu">
@@ -121,24 +118,7 @@
       <topic>/imu</topic>
       <visualize>true</visualize>
-    </sensor>
-  </gazebo>
-  <gazebo reference="camera_link">
-    <sensor name="camera" type="camera">
-      <topic>/camera/image_raw</topic>
-      <update_rate>30</update_rate>
-      <camera>
-        <horizontal_fov>1.3962634</horizontal_fov>
-        <image>
-          <width>640</width>
-          <height>480</height>
-          <format>R8G8B8</format>
-        </image>
-        <clip>
-          <near>0.02</near>
-          <far>300</far>
-        </clip>
-      </camera>
-      <always_on>1</always_on>
-      <visualize>true</visualize>
+      <plugin filename="gz-sim-imu-system"
+              name="gz::sim::systems::Imu">
+      </plugin>
     </sensor>
   </gazebo>

Commit message: Lowered the com, increased the wheel base, increased the wideth of the bot and added friction on the world.

File: install/self_balancing_bot/share/self_balancing_bot/urdf/robot.urdf.xacro (robot description, xacro)
@@ -3,10 +3,10 @@
        xmlns:xacro="http://www.ros.org/wiki/xacro">
   <xacro:property name="wheel_radius" value="0.05"/>
-  <xacro:property name="wheel_width" value="0.02"/>
+  <xacro:property name="wheel_width" value="0.04"/>
   <xacro:property name="wheel_mass" value="0.1"/>
   <xacro:property name="bot_mass" value="0.2"/>
   <xacro:property name="bot_chassis_mass" value="0.6"/>
   <xacro:property name="bot_height" value="0.25"/>
-  <xacro:property name="bot_length" value="0.15"/>
+  <xacro:property name="bot_length" value="0.17"/>
   <xacro:property name="bot_width" value="0.1"/>
   <!--Inertia Macros-->
@@ -86,8 +86,8 @@
                        y="${bot_width}"
                        z="${bot_height}"
-                       cz="0.235"/>
+                       cz="0.225"/>
   </link>
-  <xacro:wheel name="left" x_offset="0" y_offset="${0.06}"/>
-  <xacro:wheel name="right" x_offset="0" y_offset="${-0.06}"/>
+  <xacro:wheel name="left" x_offset="0" y_offset="${0.08}"/>
+  <xacro:wheel name="right" x_offset="0" y_offset="${-0.08}"/>
   <!--Dummy Base Footprint-->
   <link name="base_footprint"/>
@@ -103,5 +103,5 @@
       <left_joint>left_wheel_joint</left_joint>
       <right_joint>right_wheel_joint</right_joint>
-      <wheel_separation>${2 * 0.06}</wheel_separation>
+      <wheel_separation>${2 * 0.08}</wheel_separation>
       <wheel_radius>${wheel_radius}</wheel_radius>
       <odom_publish_frequency>50</odom_publish_frequency>
